File: FlipFlops/FlipFlops.sch (KiCad schematic (older format))
At the start: 5 parts, among them U1 74LS08, U2 74LS08, U3 74LS02, U4 74LS04

Commit message: update MSFF for waveform analysis
Parts:
- added U?: JK_MS, symbol 00TJR:JK_MS
- added U?: SR_Latch, symbol 00TJR:SR_Latch
- U?: symbol 00TJR:JK_MS -> FlipFlops-rescue:JK_MS-00TJR
Connections:
- net S0: now reaches U2.8, U3.2
- net R0: now reaches U2.11, U3.6
- net J~(Q1): now reaches U1.8, U2.9
- net K(Q1): now reaches U1.11, U2.13
- net S1: now reaches U2.6, U3.12
- net R1: now reaches U2.3, U3.8
- net C renamed Clk
- net Q renamed Q0
- net Q0: no longer U1.13, U3.10, U3.11
- net ~C renamed ~Clk
- net ~Q renamed ~Q0
- net ~Q0: no longer U1.9, U3.13, U3.9
- new net Q1: U1.13, U3.10, U3.11
- new net ~Q1: U1.9, U3.13, U3.9
Other:
- moved on the sheet: U1C, U1D

Commit message: MMFF snip ready
Parts:
- added U? (x4): 74LS02, symbol 74xx:74LS02
- added U?: 74LS04, symbol 74xx:74LS04
- added U? (x6): 74LS08, symbol 74xx:74LS08
Connections:
- net Clk: now also U?.10, U?.12, U?.5
- net J: now also U?.10
- net J~(Q1): now also U?.8, U?.9
- net K: now also U?.12
- net K(Q1): now also U?.11, U?.13
- net Q0: now also U?.3, U?.4, U?.5
- net Q1: now also U?.10, U?.11, U?.13
- net R0: now also U?.11, U?.6
- net R1: now also U?.3, U?.8
- net S0: now also U?.2, U?.8
- net S1: now also U?.12, U?.6
- net ~Clk: now also U?.2, U?.4, U?.6
- net ~Q0: now also U?.1, U?.1, U?.5
- net ~Q1: now also U?.13, U?.9, U?.9
